File: Sofle_Slim/PCB/SofleKeyboard.kicad_pcb (KiCad board)
At the start: 2 copper layers, 143.4 x 111.8 mm, 102 parts, among them J1 USB_C_Receptacle_USB2.0_14P, J2 4PIN, J3 OLED, P1 i2c_pin, P2 i2c_pin, SW1 SW_PUSH_LED, SW10 SW_PUSH_LED, SW11 SW_PUSH_LED, SW12 SW_PUSH_LED, SW13 SW_PUSH_LED, SW14 SW_PUSH_LED, SW15 SW_PUSH_LED, SW16 SW_PUSH_LED, SW17 SW_PUSH_LED, SW18 SW_PUSH_LED, SW19 SW_PUSH_LED, SW2 SW_PUSH_LED, SW20 SW_PUSH_LED, SW21 SW_PUSH_LED, SW22 SW_PUSH_LED, SW23 SW_PUSH_LED, SW24 SW_PUSH_LED, SW25 Rotary_Encoder_Switch, SW26 SW_PUSH_LED, SW27 SW_PUSH_LED, SW28 SW_PUSH_LED, SW29 SW_PUSH_LED, SW3 SW_PUSH_LED, SW30 SW_PUSH_LED, SW4 SW_PUSH_LED, SW5 SW_PUSH_LED, SW6 SW_PUSH_LED, SW7 SW_PUSH_LED, SW8 SW_PUSH_LED, SW9 SW_PUSH_LED, U2 ATmega32U4-A, Y1 16MHz

Commit message: PCB work in progress
Parts:
- J1: footprint Connector_USB:USB_C_Receptacle_GCT_USB4135-GF-A_6P_TopMnt_Horizontal -> Connector_USB:USB_C_Receptacle_Molex_105450-0101
- R8: value 10k -> 10K
- moved J1 38.9 mm to (99.5, 44.8)
Routing:
- net col0: track 336.6 -> 183.9 mm, vias 7 -> 6
- net col1: track 317.4 -> 182.0 mm, vias 9 -> 8
- net col2: track 304.4 -> 188.3 mm, vias 9 -> 8
- net GND: track 1121.9 -> 1016.6 mm, vias 44 -> 39
- net col3: track 290.9 -> 195.8 mm, vias 9 -> 8
- net col4: track 288.6 -> 209.7 mm, vias 7 -> 6
- net SW25A: track 201.0 -> 137.9 mm, vias 5 -> 4
- net RESET: track 51.2 -> 1.87 mm
- net DATA: track 48.7 -> 4.40 mm, vias 3 -> 1
- net ENCA: track 69.0 -> 25.6 mm, vias 1 -> 0
- net SDA: track 57.5 -> 14.7 mm, vias 4 -> 0
- net +5V: track 48.4 -> 15.1 mm, vias 2 -> 1
- net SCL: track 49.6 -> 17.2 mm, vias 3 -> 1
- net ENCB: track 73.9 -> 45.6 mm, vias 1 -> 0
- net row4: track 189.5 -> 168.1 mm, vias 8 -> 7
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Other:
- board size 143.4 x 111.8 mm -> 143.3 x 111.3 mm
